File: hardware/src/BDCSC.kicad_sch (KiCad schematic)
At the start: 40 parts, among them J1 Conn_02x03_Odd_Even, J10 Conn_02x01, J11 Conn_02x01, J2 Conn_02x03_Odd_Even, J3 Conn_01x05, J4 Conn_02x01, J5 Conn_02x01, J6 Conn_01x06_Pin, J7 Conn_02x01, J8 Conn_01x03, J9 Conn_02x01, U1 INA180A3, U2 LM358, U3 DRV8870DDA, U4 PY32F003F1xPx

Commit message: cleanup in preparation for hardware
Parts:
- added C12: 100uF, Capacitor_Tantalum_SMD:CP_EIA-3528-21_Kemet-B, symbol Device:C_Polarized_Small
- added J12: Conn_02x04_Odd_Even, Connector_PinHeader_2.54mm:PinHeader_2x04_P2.54mm_Vertical, symbol Connector_Generic:Conn_02x04_Odd_Even
- J1, J2: footprint Connector_PinSocket_2.54mm:PinSocket_2x03_P2.54mm_Vertical -> Connector_PinHeader_2.54mm:PinHeader_2x03_P2.54mm_Vertical
- J6: footprint Connector_PinSocket_2.54mm:PinSocket_1x06_P2.54mm_Vertical -> Connector_PinHeader_2.54mm:PinHeader_1x06_P2.54mm_Vertical
- J8: footprint Connector_PinSocket_2.54mm:PinSocket_1x03_P2.54mm_Vertical -> Connector_PinHeader_2.54mm:PinHeader_1x03_P2.54mm_Vertical
- R1: value .68R -> .680R
- U1: value INA180A3 -> INA180A1
Connections:
- net +5V: now also C12.1
- net Debug Pin 1: now also J12.1 (Pin_1)
- net Debug Pin 2: now also J12.3 (Pin_3)
- net Debug Pin 3: now also J12.5 (Pin_5)
- net Debug Pin 4: now also J12.7 (Pin_7)
- net GND: now also C12.2, J12.2 (Pin_2), J12.4 (Pin_4), J12.6 (Pin_6), J12.8 (Pin_8)
- net at C7.2, R7.2: now also J2.4 (Pin_4); no longer J2.3 (Pin_3)
- net at C8.2, R8.2: now also J2.6 (Pin_6); no longer J2.5 (Pin_5)
- net at J1.1 (Pin_1): now also J1.3 (Pin_3), J1.5 (Pin_5), J2.1 (Pin_1), J2.3 (Pin_3), J2.5 (Pin_5), U2.2 (-); no longer C2.2
- net at C4.2: now also J1.4 (Pin_4); no longer J1.3 (Pin_3)
- net at C5.2: now also J1.6 (Pin_6); no longer J1.5 (Pin_5)
- net at C6.2, R6.2: now also J2.2 (Pin_2); no longer J2.1 (Pin_1)
- new net: C2.2, J1.2 (Pin_2)
- no-connect marks 3 -> 4
Other:
- note added: "0.350A * 0.680R * 20V/V = 4.76V"
- title: Side Panel -> BDCSC

Commit message: Updated dev board and cad model
Parts:
- removed C2: 470nF, Capacitor_SMD:C_0805_2012Metric, symbol Device:C
- removed C4: 180nF, Capacitor_SMD:C_0805_2012Metric, symbol Device:C
- removed C5: 91nF, Capacitor_SMD:C_0805_2012Metric, symbol Device:C
- removed C6: 24nF, Capacitor_SMD:C_0805_2012Metric, symbol Device:C
- removed C7: 16nF, Capacitor_SMD:C_0805_2012Metric, symbol Device:C
- removed C8: 12nF, Capacitor_SMD:C_0805_2012Metric, symbol Device:C
- removed J1, J2: Conn_02x03_Odd_Even, Connector_PinHeader_2.54mm:PinHeader_2x03_P2.54mm_Vertical, symbol Connector_Generic:Conn_02x03_Odd_Even
- removed J11: Conn_02x01, Connector_PinHeader_2.54mm:PinHeader_2x01_P2.54mm_Vertical, symbol Connector_Generic:Conn_02x01
- removed R2, R4, R5, R6, R7: 3K3, Resistor_SMD:R_0805_2012Metric, symbol Device:R
- removed U1: INA180A1, Package_TO_SOT_SMD:SOT-23-5, symbol Amplifier_Current:INA180A3
- added J1: Conn_02x01, Connector_PinHeader_2.54mm:PinHeader_2x01_P2.54mm_Vertical, symbol Connector_Generic:Conn_02x01
- added J11: Conn_01x04_Pin, Connector_PinHeader_2.54mm:PinHeader_1x04_P2.54mm_Vertical, symbol Connector:Conn_01x04_Pin
- added J2: Barrel_Jack_Switch, Connector_BarrelJack:BarrelJack_CLIFF_FC681465S_SMT_Horizontal, symbol Connector:Barrel_Jack_Switch
- added R10, R11, R9: 20K, Resistor_SMD:R_0805_2012Metric, symbol Device:R
- added TP1, TP10, TP11, TP12, TP13, TP14, TP2, TP3, TP4, TP5, TP6, TP7, TP8, TP9: TestPoint, TestPoint:TestPoint_Keystone_5000-5004_Miniature, symbol Connector:TestPoint
- added U5: INA181, Package_TO_SOT_SMD:SOT-23-6, symbol Amplifier_Current:INA181
- J3: footprint Connector_PinHeader_2.54mm:PinHeader_1x05_P2.54mm_Vertical -> Connector_PinHeader_2.54mm:PinHeader_1x05_P2.54mm_Horizontal
- J6: footprint Connector_PinHeader_2.54mm:PinHeader_1x06_P2.54mm_Vertical -> Connector_PinHeader_2.54mm:PinHeader_1x06_P2.54mm_Horizontal
- R1: value .680R -> 0.15R
- R8: value 3K3 -> 20K; now not fitted
- renumbered R3 to R12, R9 to R2, R10 to R3, R11 to R4, R12 to R5, R14 to R6, R13 to R7
Connections:
- net +12V: now also J2.1
- net +5V: now also J3.1 (Pin_1), U3.4 (VREF), U5.6 (V+); no longer J3.5 (Pin_5)
- net Debug Pin 1: now also TP10.1
- net Debug Pin 2: now also TP11.1
- net Debug Pin 3: now also U4.14 (PB7), TP12.1; no longer U4.13 (PB6)
- net Debug Pin 4: now also U4.13 (PB6), TP13.1; no longer U4.14 (PB7)
- net ENC_IN_A: now also U4.4 (PA5), TP5.1; no longer U4.5 (PA6)
- net ENC_IN_B: now also U4.5 (PA6), TP6.1; no longer U4.4 (PA5)
- net GND: now also U3.7 (ISEN), J2.2, J2.3, R11.1, U5.2 (GND); no longer R1.2
- net Motor IN_A: now also TP7.1
- net Motor IN_B: now also TP8.1
- net SWC: now also J3.4 (Pin_4); no longer J3.2 (Pin_2)
- net SWD: now also J3.2 (Pin_2); no longer J3.4 (Pin_4)
- net ~{RST}: now also J3.5 (Pin_5); no longer J3.1 (Pin_1)
- net at C10.1, R4.1, R6.1: now also U2.3 (+); no longer U2.5 (+)
- net Diff Amp Out: now reaches J7.1 (Pin_1)
- net Diff Amp Out: now also R7.2, U2.1, TP9.1
- net at R1.1: now also U3.6 (OUT1), TP3.1, U5.4 (-); no longer U3.7 (ISEN)
- net at U2.2 (-): now also R5.1, R7.1
- net at R8.2: now also J11.2 (Pin_2)
- net Diff Amp In: now reaches R4.2, R5.2
- net Diff Amp In: now also J4.1 (Pin_1); no longer J9.2 (Pin_2)
- net MOTOR_N renamed Motor +
- net Motor +: now also J6.1 (Pin_1), TP1.1; no longer J6.6 (Pin_6)
- removed net MOTOR_P: J6.1 (Pin_1), U3.6 (OUT1)
- removed net MOTOR_PULSES: J4.1 (Pin_1), R7.2, U2.7
- net MOTOR_PULSE_COMP renamed Motor Current
- net Motor Current: now also TP4.1, U5.1; no longer U4.2 (PA3)
- net bpf_in renamed Motor Pulses µC
- net Motor Pulses µC: now also U4.2 (PA3)
- removed net bpf_out: J9.1 (Pin_1), R8.1, U2.1
- new net: J1.2 (Pin_2), U5.5 (REF)
- new net: R10.2, R9.1, U2.6 (-)
- new net: J11.3 (Pin_3), R9.2
- new net: J11.1 (Pin_1), R11.2, R8.1, U2.5 (+)
- new net: J11.4 (Pin_4), R10.1, TP14.1, U2.7
- new net +2V5: J1.1 (Pin_1), J10.2 (Pin_2), J9.2 (Pin_2)
- new net Diff Amp Vreff: J9.1 (Pin_1), R6.2
- new net Motor -: J6.6 (Pin_6), R1.2, TP2.1, U5.3 (+)
Other:
- note added: "GAIN: 50 Small phace shift itroduced in AMP+ by C10"
- note added: "Motor Controller + CSA"
- note added: "Power"
- note added: "R1 = 0.833A * 0.150R * 20V/V = 2.5V"
- note added: "Spare Amplifier"
- note removed: "0.350A * 0.680R * 20V/V = 4.76V"
- note removed: "102Hz"
- note removed: "2000Hz"
- note removed: "268Hz"
- note removed: "3000Hz"
- note removed: "4000Hz"
- note removed: "530Hz"
- note removed: "Active Band Pass filter"
- note removed: "Low frequency cutoff"
- note removed: "Motor Controller"
- moved on the sheet: C10, C12, C3, C9, J10, J12, J6, J8, R1, R2, R3, R4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
